File: PCB_N2A/PCB_N2A.kicad_pcb (KiCad board)
At the start: 2 copper layers, 81 x 90 mm, 42 parts, among them J1 Conn_01x08, J2 Teclado, J3 LCD, J4 SENS, Q1 BC547, U1 68HC11_PLCC, U2 MAX232CPE, U3 24LC65, U4 MAX703, U5 DS1302+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

Commit message: wip
Other:
- net class Default removed
